File: KiCAD/CarteMereRobobeer/CarteMereRobobeer.kicad_pcb (KiCad board)
At the start: 2 copper layers, 114 x 88 mm, 93 parts, among them J1 Conn_01x01_Male, J2 Conn_01x01_Male, J3 Conn_01x01_Male, J4 Conn_01x01_Male, U2 MC34063ADR2G, U4 MC34063ADR2G, U5 Quartz, U6 STM32F103RCTx

Commit message: updated KiCAD
Motherboard
Routing:
- net GND: track 276.7 -> 304.2 mm, vias 32 -> 33
- net PINCE_PWM: track 71.5 -> 61.5 mm
- net USART2_TX: track 127.7 -> 136.6 mm
- net TOF_I2C_SDA: track 80.8 -> 78.0 mm
- net USART2_RX: track 130.2 -> 128.2 mm
- net MOTOR_2_PWM_IN2: track 69.0 -> 67.2 mm
- net NRST: track 103.0 -> 101.2 mm
- net MOTOR_2_A: track 36.8 -> 35.1 mm
- net Net-(D7-Pad2): track 19.6 -> 20.9 mm
- net Alim_Rasp: track 72.9 -> 71.8 mm
- net USER_BTN: track 78.5 -> 77.4 mm
- net /Driver_moteur_gauche/RS_Motor2: track 37.3 -> 36.5 mm
- net CURRENT_SENSOR_2: track 88.2 -> 89.0 mm
- net +3.3V: track 180.1 -> 179.3 mm
- net BDT4: track 75.7 -> 74.9 mm
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
Commit message: update PCB
Routing:
- net BDT4: track 74.9 -> 55.9 mm
- net BDT3: track 81.2 -> 62.8 mm
- net Net-(D7-Pad2): track 20.9 -> 24.6 mm
- net Net-(BDT1-Pad2): track 13.9 -> 16.3 mm
- net GND: track 304.2 -> 302.2 mm
- net SYS_JTCK-SWCLK: track 54.1 -> 55.8 mm
- net BDT1: track 63.8 -> 62.3 mm
- net MOTOR_2_PWM_IN2: track 67.2 -> 65.8 mm
- net BDT2: track 63.5 -> 62.4 mm
- net USART2_TX: track 136.6 -> 135.5 mm
- net LED4: track 27.1 -> 26.1 mm
- net MOTOR_1_ENCODER_A: track 96.0 -> 97.0 mm
- net MOTOR_2_ENCODER_B: track 66.5 -> 67.4 mm
- net +7.5V: track 173.2 -> 172.3 mm
- net MOTOR_2_B: track 26.4 -> 27.2 mm
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
Commit message: update PCB
Routing:
- net TOF_Interrupt: track 84.2 -> 87.2 mm
- net TOF_XSHUT: track 82.1 -> 82.8 mm
- net MOTOR_1_ENCODER_A: track 97.0 -> 96.8 mm, vias 2 -> 0
Changed lines of the file:
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@@
       (drillshape 0)
       (scaleselection 1)
-      (outputdirectory "")
+      (outputdirectory "Gerber/")
     )
   )
@@
   (segment (start 158.75 93.175) (end 158.75 94.27556) (width 0.3) (layer "F.Cu") (net 4))
   (segment (start 187.9125 81.655) (end 187.9825 81.585) (width 0.6) (layer "F.Cu") (net 4))
-  (segment (start 150 66) (end 150.5 65.5) (width 0.6) (layer "F.Cu") (net 4))
   (segment (start 179.2 55) (end 179.2 57.8) (width 0.6) (layer "F.Cu") (net 4))
   (segment (start 105.12 48.3625) (end 103.344122 48.3625) (width 0.6) (layer "F.Cu") (net 4))
@@
   (segment (start 150.5 115) (end 150 115.5) (width 0.6) (layer "F.Cu") (net 4))
   (segment (start 166.075 60.3) (end 169.9 60.3) (width 0.6) (layer "F.Cu") (net 4))
+  (segment (start 150 66) (end 150.721398 65.278602) (width 0.6) (layer "F.Cu") (net 4))
   (segment (start 113.155 96.46) (end 113.195 96.5) (width 0.6) (layer "F.Cu") (net 4))
   (segment (start 153 113.38) (end 153 115) (width 0.6) (layer "F.Cu") (net 4))
@@
   (via (at 145 94.5) (size 1) (drill 0.6) (layers "F.Cu" "B.Cu") (net 4))
   (via (at 119.5 108.799001) (size 1) (drill 0.6) (layers "F.Cu" "B.Cu") (net 4))
-  (via (at 150.5 65.5) (size 1) (drill 0.6) (layers "F.Cu" "B.Cu") (net 4))
+  (via (at 150.721398 65.278602) (size 1) (drill 0.6) (layers "F.Cu" "B.Cu") (net 4))
   (via (at 163.2 83.7) (size 0.8) (drill 0.4) (layers "F.Cu" "B.Cu") (net 4))
   (via (at 159.009524 94.535084) (size 0.8) (drill 0.4) (layers "F.Cu" "B.Cu") (net 4))
@@
   (segment (start 153.25 81.825) (end 153.25 80.437197) (width 0.3) (layer "F.Cu") (net 55))
   (via (at 151.1 74.5) (size 0.8) (drill 0.4) (layers "F.Cu" "B.Cu") (net 55))
-  (segment (start 148 67.793598) (end 148 71.4) (width 0.5) (layer "B.Cu") (net 55))
-  (segment (start 98.77 59.5) (end 139.706402 59.5) (width 0.5) (layer "B.Cu") (net 55))
-  (segment (start 139.706402 59.5) (end 148 67.793598) (width 0.5) (layer "B.Cu") (net 55))
-  (segment (start 148 71.4) (end 151.1 74.5) (width 0.5) (layer "B.Cu") (net 55))
   (segment (start 91.5 52.23) (end 98.77 59.5) (width 0.5) (layer "B.Cu") (net 55))
+  (segment (start 140.1 59.5) (end 148 67.4) (width 0.5) (layer "B.Cu") (net 55))
+  (segment (start 148 67.4) (end 148 71.4) (width 0.5) (layer "B.Cu") (net 55))
+  (segment (start 98.77 59.5) (end 140.1 59.5) (width 0.5) (layer "B.Cu") (net 55))
+  (segment (start 148 71.4) (end 151.1 74.5) (width 0.5) (layer "B.Cu") (net 55))
   (segment (start 155.25 81.825) (end 155.25 77.779977) (width 0.3) (layer "F.Cu") (net 56))
   (segment (start 152.9 75.429977) (end 152.9 74.9) (width 0.3) (layer "F.Cu") (net 56))
   (segment (start 155.25 77.779977) (end 152.9 75.429977) (width 0.3) (layer "F.Cu") (net 56))
   (via (at 152.9 74.9) (size 0.8) (drill 0.4) (layers "F.Cu" "B.Cu") (net 56))
-  (segment (start 140 58) (end 152.9 70.9) (width 0.5) (layer "B.Cu") (net 56))
-  (segment (start 99.81 58) (end 140 58) (width 0.5) (layer "B.Cu") (net 56))
   (segment (start 91.5 49.69) (end 99.81 58) (width 0.5) (layer "B.Cu") (net 56))
-  (segment (start 152.9 70.9) (end 152.9 74.9) (width 0.5) (layer "B.Cu") (net 56))
+  (segment (start 141.2 58) (end 152.9 69.7) (width 0.5) (layer "B.Cu") (net 56))
+  (segment (start 99.81 58) (end 141.2 58) (width 0.5) (layer "B.Cu") (net 56))
+  (segment (start 152.9 69.7) (end 152.9 74.9) (width 0.5) (layer "B.Cu") (net 56))
   (segment (start 155.75 76.95) (end 155.1 76.3) (width 0.3) (layer "F.Cu") (net 57))
   (segment (start 155.75 81.825) (end 155.75 76.95) (width 0.3) (layer "F.Cu") (net 57))
   (via (at 155.1 76.3) (size 0.8) (drill 0.4) (layers "F.Cu" "B.Cu") (net 57))
-  (segment (start 91.5 47.15) (end 100.791224 56.441224) (width 0.5) (layer "B.Cu") (net 57))
-  (segment (start 139.941224 56.441224) (end 155.1 71.6) (width 0.5) (layer "B.Cu") (net 57))
-  (segment (start 100.791224 56.441224) (end 139.941224 56.441224) (width 0.5) (layer "B.Cu") (net 57))
-  (segment (start 155.1 71.6) (end 155.1 76.3) (width 0.5) (layer "B.Cu") (net 57))
+  (segment (start 155.1 66.5) (end 145.041224 56.441224) (width 0.5) (layer "B.Cu") (net 57))
+  (segment (start 155.1 76.3) (end 155.1 66.5) (width 0.5) (layer "B.Cu") (net 57))
+  (segment (start 145.041224 56.441224) (end 100.791224 56.441224) (width 0.5) (layer "B.Cu") (net 57))
+  (segment (start 100.791224 56.441224) (end 91.5 47.15) (width 0.5) (layer "B.Cu") (net 57))
   (segment (start 90.4 102.67) (end 90.4 101.632943) (width 0.3) (layer "F.Cu") (net 58))
   (segment (start 100.4 92.6) (end 110.4 92.6) (width 0.4) (layer "F.Cu") (net 58))
-  (segment (start 159 78.5) (end 158.75 78.75) (width 0.3) (layer "F.Cu") (net 58))
   (segment (start 147.85 73.7) (end 148.65 72.9) (width 0.4) (layer "F.Cu") (net 58))
   (segment (start 90.4 101.632943) (end 91.643443 100.3895) (width 0.3) (layer "F.Cu") (net 58))
   (segment (start 140.9 73.7) (end 147.85 73.7) (width 0.4) (layer "F.Cu") (net 58))
   (segment (start 111.3 91.7) (end 133.3 91.7) (width 0.4) (layer "F.Cu") (net 58))
-  (segment (start 155.7 72.9) (end 156.9 74.1) (width 0.4) (layer "F.Cu") (net 58))
+  (segment (start 158.75 75.95) (end 158.75 81.825) (width 0.3) (layer "F.Cu") (net 58))
   (segment (start 133.900499 80.699501) (end 140.9 73.7) (width 0.4) (layer "F.Cu") (net 58))
   (segment (start 92.6105 100.3895) (end 100.4 92.6) (width 0.4) (layer "F.Cu") (net 58))
   (segment (start 110.4 92.6) (end 111.3 91.7) (width 0.4) (layer "F.Cu") (net 58))
   (segment (start 91.643443 100.3895) (end 92.6105 100.3895) (width 0.3) (layer "F.Cu") (net 58))
+  (segment (start 155.7 72.9) (end 158.75 75.95) (width 0.3) (layer "F.Cu") (net 58))
   (segment (start 148.65 72.9) (end 155.7 72.9) (width 0.4) (layer "F.Cu") (net 58))
   (segment (start 133.900499 91.099501) (end 133.900499 80.699501) (width 0.4) (layer "F.Cu") (net 58))
   (segment (start 92 104.27) (end 90.4 102.67) (width 0.3) (layer "F.Cu") (net 58))
-  (segment (start 158.75 78.75) (end 158.75 81.825) (width 0.3) (layer "F.Cu") (net 58))
   (segment (start 133.3 91.7) (end 133.900499 91.099501) (width 0.4) (layer "F.Cu") (net 58))
-  (via (at 159 78.5) (size 0.8) (drill 0.4) (layers "F.Cu" "B.Cu") (net 58))
-  (via (at 156.9 74.1) (size 0.8) (drill 0.4) (layers "F.Cu" "B.Cu") (net 58))
-  (segment (start 159 78.5) (end 158.1 77.6) (width 0.5) (layer "B.Cu") (net 58))
-  (segment (start 158.1 77.6) (end 158.1 75.3) (width 0.5) (layer "B.Cu") (net 58))
-  (segment (start 158.1 75.3) (end 156.9 74.1) (width 0.5) (layer "B.Cu") (net 58))
   (segment (start 101.432081 93.5) (end 111.7 93.5) (width 0.4) (layer "F.Cu") (net 59))
   (segment (start 141.2 74.7) (end 147.9 74.7) (width 0.4) (layer "F.Cu") (net 59))
