File: KiCAD/Couleur/Couleur.kicad_pcb (KiCad board)
At the start: 2 copper layers, 25 x 9.5 mm, 7 parts, among them IC1 VEML3328, J1 Conn_01x04_Male

Commit message: update PCB
Routing:
- net COLOR_I2C_SDA: track 9.16 -> 8.30 mm
- net COLOR_I2C_SCL: track 9.05 -> 8.26 mm
- net +3.3V: track 26.3 -> 25.7 mm
Changed lines of the file:
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@@
   )
   (gr_rect (start 75.5 75) (end 100.5 84.5) (layer "Edge.Cuts") (width 0.1) (fill none))
-  (segment (start 86.15 80.85) (end 86 81) (width 0.25) (layer "F.Cu") (net 1))
+  (segment (start 86.15 80.85) (end 86 81) (width 0.4) (layer "F.Cu") (net 1))
+  (segment (start 86.275 80.85) (end 84.2 78.775) (width 0.4) (layer "F.Cu") (net 1))
   (segment (start 86.275 80.85) (end 86.15 80.85) (width 0.25) (layer "F.Cu") (net 1))
-  (segment (start 87.05 80.85) (end 86.275 80.85) (width 0.25) (layer "F.Cu") (net 1))
-  (segment (start 86.5 82.5) (end 87.5925 82.5) (width 0.25) (layer "F.Cu") (net 1))
-  (segment (start 86 82) (end 86.5 82.5) (width 0.25) (layer "F.Cu") (net 1))
-  (segment (start 86.275 80.85) (end 84.2 78.775) (width 0.25) (layer "F.Cu") (net 1))
-  (segment (start 84.2 78.775) (end 84.2 76.5) (width 0.25) (layer "F.Cu") (net 1))
-  (segment (start 86 81) (end 86 82) (width 0.25) (layer "F.Cu") (net 1))
-  (segment (start 84.2 76.5) (end 84.2 77.3) (width 0.25) (layer "B.Cu") (net 1))
-  (segment (start 89.9075 82.5) (end 84.5 82.5) (width 0.25) (layer "B.Cu") (net 1))
-  (segment (start 83 82) (end 83.5 82.5) (width 0.25) (layer "B.Cu") (net 1))
-  (segment (start 85 82) (end 84.5 82.5) (width 0.25) (layer "B.Cu") (net 1))
-  (segment (start 84.2 77.3) (end 83 78.5) (width 0.25) (layer "B.Cu") (net 1))
-  (segment (start 85 80.9075) (end 85 82) (width 0.25) (layer "B.Cu") (net 1))
-  (segment (start 83 78.5) (end 83 82) (width 0.25) (layer "B.Cu") (net 1))
-  (segment (start 84.5 82.5) (end 83.5 82.5) (width 0.25) (layer "B.Cu") (net 1))
-  (segment (start 91.5 80.9075) (end 89.9075 82.5) (width 0.25) (layer "B.Cu") (net 1))
-  (segment (start 91.82 78.755) (end 91.82 76.5) (width 0.25) (layer "F.Cu") (net 2))
-  (segment (start 89.9375 82.0625) (end 89.9375 81) (width 0.25) (layer "F.Cu") (net 2))
-  (segment (start 89.9375 81) (end 89.7875 80.85) (width 0.25) (layer "F.Cu") (net 2))
-  (segment (start 89.7875 80.85) (end 89.725 80.85) (width 0.25) (layer "F.Cu") (net 2))
-  (segment (start 89.5 82.5) (end 89.9375 82.0625) (width 0.25) (layer "F.Cu") (net 2))
-  (segment (start 88.95 80.85) (end 89.725 80.85) (width 0.25) (layer "F.Cu") (net 2))
-  (segment (start 88.4075 82.5) (end 89.5 82.5) (width 0.25) (layer "F.Cu") (net 2))
+  (segment (start 87.05 80.85) (end 86.275 80.85) (width 0.4) (layer "F.Cu") (net 1))
+  (segment (start 86.5 82.5) (end 87.5925 82.5) (width 0.4) (layer "F.Cu") (net 1))
+  (segment (start 86 82) (end 86.5 82.5) (width 0.4) (layer "F.Cu") (net 1))
+  (segment (start 84.2 78.775) (end 84.2 76.5) (width 0.4) (layer "F.Cu") (net 1))
+  (segment (start 86 81) (end 86 82) (width 0.4) (layer "F.Cu") (net 1))
+  (segment (start 84.5 82.5) (end 83 81) (width 0.5) (layer "B.Cu") (net 1))
+  (segment (start 89.9075 82.5) (end 84.5 82.5) (width 0.5) (layer "B.Cu") (net 1))
+  (segment (start 83 81) (end 83 78.4) (width 0.5) (layer "B.Cu") (net 1))
+  (segment (start 84.2 77.2) (end 84.1 77.3) (width 0.25) (layer "B.Cu") (net 1))
+  (segment (start 83 78.4) (end 84.1 77.3) (width 0.5) (layer "B.Cu") (net 1))
+  (segment (start 85 82) (end 84.5 82.5) (width 0.5) (layer "B.Cu") (net 1))
+  (segment (start 84.2 76.5) (end 84.2 77.2) (width 0.5) (layer "B.Cu") (net 1))
+  (segment (start 85 80.9075) (end 85 82) (width 0.5) (layer "B.Cu") (net 1))
+  (segment (start 91.5 80.9075) (end 89.9075 82.5) (width 0.5) (layer "B.Cu") (net 1))
+  (segment (start 91.82 78.755) (end 91.82 76.5) (width 0.4) (layer "F.Cu") (net 2))
+  (segment (start 89.9375 82.0625) (end 89.9375 81) (width 0.4) (layer "F.Cu") (net 2))
+  (segment (start 89.9375 81) (end 89.7875 80.85) (width 0.4) (layer "F.Cu") (net 2))
+  (segment (start 89.7875 80.85) (end 89.725 80.85) (width 0.4) (layer "F.Cu") (net 2))
+  (segment (start 89.5 82.5) (end 89.9375 82.0625) (width 0.4) (layer "F.Cu") (net 2))
+  (segment (start 88.95 80.85) (end 89.725 80.85) (width 0.4) (layer "F.Cu") (net 2))
+  (segment (start 88.4075 82.5) (end 89.5 82.5) (width 0.4) (layer "F.Cu") (net 2))
   (segment (start 89 80.9) (end 88.95 80.85) (width 0.25) (layer "F.Cu") (net 2))
-  (segment (start 89.725 80.85) (end 91.82 78.755) (width 0.25) (layer "F.Cu") (net 2))
-  (segment (start 90.13 79.245) (end 90.13 77.35) (width 0.25) (layer "F.Cu") (net 3))
-  (segment (start 88.95 80.15) (end 89.225 80.15) (width 0.25) (layer "F.Cu") (net 3))
-  (segment (start 89.225 80.15) (end 90.13 79.245) (width 0.25) (layer "F.Cu") (net 3))
-  (segment (start 90.13 77.35) (end 89.28 76.5) (width 0.25) (layer "F.Cu") (net 3))
-  (segment (start 91.5 80.0925) (end 91.5 78.72) (width 0.25) (layer "B.Cu") (net 3))
-  (segment (start 91.5 78.72) (end 89.28 76.5) (width 0.25) (layer "B.Cu") (net 3))
-  (segment (start 86.352112 80.15) (end 85.89 79.687888) (width 0.25) (layer "F.Cu") (net 4))
-  (segment (start 86.6 80.15) (end 86.352112 80.15) (width 0.25) (layer "F.Cu") (net 4))
-  (segment (start 85.89 77.35) (end 86.74 76.5) (width 0.25) (layer "F.Cu") (net 4))
-  (segment (start 85.89 79.687888) (end 85.89 77.35) (width 0.25) (layer "F.Cu") (net 4))
-  (segment (start 85 79.5) (end 86 78.5) (width 0.25) (layer "B.Cu") (net 4))
-  (segment (start 85 80.0925) (end 85 79.5) (width 0.25) (layer "B.Cu") (net 4))
-  (segment (start 86 78.5) (end 86.5 78.5) (width 0.25) (layer "B.Cu") (net 4))
-  (segment (start 86.5 78.5) (end 86.74 78.26) (width 0.25) (layer "B.Cu") (net 4))
-  (segment (start 86.74 78.26) (end 86.74 76.5) (width 0.25) (layer "B.Cu") (net 4))
+  (segment (start 89.725 80.85) (end 91.82 78.755) (width 0.4) (layer "F.Cu") (net 2))
+  (segment (start 89.28 76.5) (end 89.28 78.62) (width 0.4) (layer "F.Cu") (net 3))
+  (segment (start 89.28 78.62) (end 89 78.9) (width 0.4) (layer "F.Cu") (net 3))
+  (segment (start 88.95 78.95) (end 89 78.9) (width 0.25) (layer "F.Cu") (net 3))
+  (segment (start 88.95 80.15) (end 88.95 78.95) (width 0.4) (layer "F.Cu") (net 3))
+  (segment (start 91.5 80.0925) (end 91.5 78.72) (width 0.5) (layer "B.Cu") (net 3))
+  (segment (start 91.5 78.72) (end 89.28 76.5) (width 0.5) (layer "B.Cu") (net 3))
+  (segment (start 86.74 79.79) (end 87.0005 80.0505) (width 0.5) (layer "F.Cu") (net 4))
+  (segment (start 86.74 76.5) (end 86.74 79.79) (width 0.5) (layer "F.Cu") (net 4))
+  (segment (start 85 79.5) (end 86 78.5) (width 0.5) (layer "B.Cu") (net 4))
+  (segment (start 85 80.0925) (end 85 79.5) (width 0.5) (layer "B.Cu") (net 4))
+  (segment (start 86 78.5) (end 86.5 78.5) (width 0.5) (layer "B.Cu") (net 4))
+  (segment (start 86.5 78.5) (end 86.74 78.26) (width 0.5) (layer "B.Cu") (net 4))
+  (segment (start 86.74 78.26) (end 86.74 76.5) (width 0.5) (layer "B.Cu") (net 4))
   (zone (net 2) (net_name "GND") (layers F&B.Cu) (hatch edge 0.508)
     (connect_pads (clearance 0.508))
